File: prod/mosaic.kicad_pcb (KiCad board)
At the start: 2 copper layers, 100 x 85 mm, 23 parts

Commit message: v0.0.1 prototypes
Routing:
- net matrix_inner_top: track 0.00 -> 141.1 mm
- net matrix_inner_home: track 0.00 -> 120.7 mm
- net thumbfan_far_home: track 0.00 -> 117.3 mm
- net matrix_inner_bottom: track 0.00 -> 99.8 mm
- net thumbfan_home_home: track 0.00 -> 96.6 mm
- net matrix_index_top: track 0.00 -> 94.2 mm
- net 3V3: track 0.00 -> 90.0 mm
- net GP8: track 0.00 -> 85.2 mm, vias 0 -> 2
- net GP9: track 0.00 -> 82.5 mm, vias 0 -> 2
- net matrix_ring_top: track 0.00 -> 78.3 mm
- net matrix_index_home: track 0.00 -> 77.3 mm
- net matrix_middle_top: track 0.00 -> 76.4 mm
- net thumbfan_near_home: track 0.00 -> 75.5 mm
- net matrix_ring_home: track 0.00 -> 63.6 mm
- net matrix_index_bottom: track 0.00 -> 61.3 mm
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- added copper zone on B.Cu, net GND
- added copper zone on F.Cu, net GND

Commit message: v0.1.0: cleaner routing for split comm traces
Routing:
- net GP8: track 85.2 -> 93.4 mm
- net GP9: track 82.5 -> 90.5 mm
- net matrix_pinky_home: track 43.3 -> 42.0 mm
- net 3V3: track 90.0 -> 91.0 mm
- net matrix_pinky_bottom: track 25.8 -> 26.6 mm
- net GND: vias 2 -> 11
Other:
- board text added: "mosaic v0.1.0"
- board text removed: "mosaic v0.0.1"
